File: arduinoToEsp32.kicad_pcb (KiCad board)
At the start: 2 copper layers, 4 parts, among them J1 Conn_01x03_Pin

Commit message: correção do esquematico
Routing:
- added copper zone on B.Cu, net GND
Changed lines of the file:
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@@
 		(pad "1" thru_hole circle
 			(at 0 0 90)
-			(size 1.6 1.6)
+			(size 2 2)
 			(drill 0.8)
 			(layers "*.Cu" "*.Mask")
@@
 		(pad "1" thru_hole circle
 			(at 0 0 90)
-			(size 1.6 1.6)
+			(size 2 2)
 			(drill 0.8)
 			(layers "*.Cu" "*.Mask")
@@
 		(pad "2" thru_hole circle
 			(at 15.24 0 90)
-			(size 1.6 1.6)
+			(size 2 2)
 			(drill 0.8)
 			(layers "*.Cu" "*.Mask")
@@
 		(pad "1" thru_hole circle
 			(at 0 0 90)
-			(size 1.6 1.6)
+			(size 2 2)
 			(drill 0.8)
 			(layers "*.Cu" "*.Mask")
@@
 		(pad "2" thru_hole circle
 			(at 15.24 0 90)
-			(size 1.6 1.6)
+			(size 2 2)
 			(drill 0.8)
 			(layers "*.Cu" "*.Mask")
@@
 			)
 		)
+	)
+	(zone
+		(net 4)
+		(net_name "GND")
+		(layer "B.Cu")
+		(hatch edge 0.5)
+		(connect_pads
+			(clearance 0.5)
+		)
+		(min_thickness 0.25)
+		(filled_areas_thickness no)
+		(fill yes
+			(thermal_gap 0.5)
+			(thermal_bridge_width 0.5)
+		)
+		(polygon
+			(pts
+				(xy 153.363855 57.359152) (xy 172.466 57.023) (xy 172.254935 85.344) (xy 153.363855 85.344)
+			)
+		)

Commit message: trilhas adicionadas
Connections:
- net Net-(J1-Pin_1) renamed +5V
Routing:
- net GND: track 0.00 -> 64.8 mm
- net Net-(1k1-Pad2): track 0.00 -> 14.6 mm
- net Net-(J1-Pin_2): track 0.00 -> 10.7 mm
- net +5V: track 0.00 -> 4.72 mm
- removed copper zone on B.Cu, net GND
Changed lines of the file:
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@@
 	)
 	(net 0 "")
-	(net 1 "Net-(J1-Pin_1)")
+	(net 1 "+5V")
 	(net 2 "Net-(1k1-Pad2)")
 	(net 3 "Net-(J1-Pin_2)")
@@
 			(remove_unused_layers no)
 			(roundrect_rratio 0.096154)
-			(net 1 "Net-(J1-Pin_1)")
+			(net 1 "+5V")
 			(pinfunction "Pin_1")
 			(pintype "passive")
@@
 			(layers "*.Cu" "*.Mask")
 			(remove_unused_layers no)
-			(net 1 "Net-(J1-Pin_1)")
+			(net 1 "+5V")
 			(pintype "passive")
 		)
@@
 		)
 	)
-	(zone
-		(net 0)
-		(net_name "")
-		(layer "B.Cu")
-		(name "Placa")
-		(hatch edge 0.5)
-		(connect_pads
-			(clearance 0)
-		)
-		(min_thickness 0.25)
-		(filled_areas_thickness no)
-		(keepout
-			(tracks not_allowed)
-			(vias not_allowed)
-			(pads not_allowed)
-			(copperpour allowed)
-			(footprints allowed)
-		)
-		(placement
-			(enabled no)
-			(sheetname "/")
-		)
-		(fill
-			(thermal_gap 0.5)
-			(thermal_bridge_width 0.5)
-		)
-		(polygon
-			(pts
-				(xy 153.363855 57.359152) (xy 172.466 57.023) (xy 172.254935 85.344) (xy 153.363855 85.344) (xy 153.363855 59.436)
-			)
-		)
-	)
-	(zone
+	(segment
+		(start 156.871 79.248)
+		(end 156.871 75.031)
+		(width 2)
+		(layer "B.Cu")
+		(net 1)
+	)
+	(segment
+		(start 156.871 75.031)
+		(end 157.226 74.676)
+		(width 2)
+		(layer "B.Cu")
+		(net 1)
+	)
+	(segment
+		(start 166.243 57.658)
+		(end 168.148 59.563)
+		(width 2)
+		(layer "B.Cu")
+		(net 2)
+	)
+	(segment
+		(start 157.226 58.547)
+		(end 159.385 56.388)
+		(width 2)
+		(layer "B.Cu")
+		(net 2)
+	)
+	(segment
+		(start 165.989 56.388)
+		(end 166.243 56.642)
+		(width 2)
+		(layer "B.Cu")
+		(net 2)
+	)
+	(segment
+		(start 157.226 59.436)
+		(end 157.226 58.547)
+		(width 2)
+		(layer "B.Cu")
+		(net 2)
+	)
+	(segment
+		(start 166.243 56.642)
+		(end 166.243 57.658)
+		(width 2)
+		(layer "B.Cu")
+		(net 2)
+	)
+	(segment
+		(start 159.385 56.388)
+		(end 165.989 56.388)
+		(width 2)
+		(layer "B.Cu")
+		(net 2)
+	)
+	(segment
+		(start 162.433 74.676)
+		(end 168.021 74.676)
+		(width 2)
+		(layer "B.Cu")
+		(net 3)
+	)
+	(segment
+		(start 161.671 79.248)
+		(end 161.671 75.438)
+		(width 2)
+		(layer "B.Cu")
+		(net 3)
+	)
+	(segment
+		(start 168.021 74.676)
+		(end 168.148 74.803)
+		(width 2)
+		(layer "B.Cu")
+		(net 3)
+	)
+	(segment
+		(start 161.671 75.438)
+		(end 162.433 74.676)
+		(width 2)
+		(layer "B.Cu")
+		(net 3)
+	)
+	(segment
+		(start 167.386 53.086)
+		(end 158.877 53.086)
+		(width 2)
+		(layer "B.Cu")
 		(net 4)
-		(net_name "GND")
-		(layer "B.Cu")
-		(hatch edge 0.5)
-		(connect_pads
-			(clearance 0.5)
-		)
-		(min_thickness 0.25)
-		(filled_areas_thickness no)
-		(fill yes
-			(thermal_gap 0.5)
-			(thermal_bridge_width 0.5)
-		)
-		(polygon
-			(pts
-				(xy 153.363855 57.359152) (xy 172.466 57.023) (xy 172.254935 85.344) (xy 153.363855 85.344)
-			)
-		)
+	)
+	(segment
+		(start 171.578602 57.786602)
+		(end 167.386 53.594)
+		(width 2)
+		(layer "B.Cu")
+		(net 4)
+	)
+	(segment
+		(start 158.877 53.086)
+		(end 153.543 58.42)
+		(width 2)
+		(layer "B.Cu")
+		(net 4)
+	)
+	(segment
+		(start 161.163 63.246)
+		(end 162.433 61.976)
+		(width 2)
+		(layer "B.Cu")
+		(net 4)
+	)
+	(segment
+		(start 167.386 53.594)
+		(end 167.386 53.086)
+		(width 2)
+		(layer "B.Cu")
+		(net 4)
+	)
+	(segment
+		(start 171.578602 79.246398)
+		(end 171.578602 57.786602)
+		(width 2)
+		(layer "B.Cu")
+		(net 4)
+	)
+	(segment
+		(start 171.069 79.248)
+		(end 171.323 79.502)
+		(width 2)
+		(layer "B.Cu")
+		(net 4)
+	)
+	(segment
+		(start 155.702 63.246)
+		(end 161.163 63.246)
+		(width 2)
+		(layer "B.Cu")
+		(net 4)
+	)
+	(segment
+		(start 166.471 79.248)
+		(end 171.069 79.248)
+		(width 2)
+		(layer "B.Cu")
+		(net 4)
+	)
+	(segment
+		(start 171.323 79.502)
+		(end 171.578602 79.246398)
+		(width 2)
+		(layer "B.Cu")
+		(net 4)
+	)
+	(segment
+		(start 153.543 61.087)
+		(end 155.702 63.246)
+		(width 2)
+		(layer "B.Cu")
+		(net 4)
+	)
+	(segment
+		(start 162.433 61.976)
+		(end 162.433 59.436)
+		(width 2)
+		(layer "B.Cu")
+		(net 4)
+	)
+	(segment
+		(start 153.543 58.42)
+		(end 153.543 61.087)
+		(width 2)
+		(layer "B.Cu")
+		(net 4)
 	)
 	(embedded_fonts no)

Commit message: finalizado
Routing:
- net GND: track 64.8 -> 15.5 mm
- added copper zone on B.Cu, net GND
Changed lines of the file:
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@@
-	)
-	(segment
-		(start 167.386 53.086)
-		(end 158.877 53.086)
-		(width 2)
-		(layer "B.Cu")
-		(net 4)
-	)
-	(segment
-		(start 171.578602 57.786602)
-		(end 167.386 53.594)
-		(width 2)
-		(layer "B.Cu")
-		(net 4)
-	)
-	(segment
-		(start 158.877 53.086)
-		(end 153.543 58.42)
-		(width 2)
-		(layer "B.Cu")
-		(net 4)
 	)
 	(segment
@@
 	)
 	(segment
-		(start 167.386 53.594)
-		(end 167.386 53.086)
-		(width 2)
-		(layer "B.Cu")
-		(net 4)
-	)
-	(segment
-		(start 171.578602 79.246398)
-		(end 171.578602 57.786602)
-		(width 2)
-		(layer "B.Cu")
-		(net 4)
-	)
-	(segment
-		(start 171.069 79.248)
-		(end 171.323 79.502)
-		(width 2)
-		(layer "B.Cu")
-		(net 4)
-	)
-	(segment
 		(start 155.702 63.246)
 		(end 161.163 63.246)
-		(width 2)
-		(layer "B.Cu")
-		(net 4)
-	)
-	(segment
-		(start 166.471 79.248)
-		(end 171.069 79.248)
-		(width 2)
-		(layer "B.Cu")
-		(net 4)
-	)
-	(segment
-		(start 171.323 79.502)
-		(end 171.578602 79.246398)
 		(width 2)
 		(layer "B.Cu")
@@
 		(net 4)
 	)
+	(zone
+		(net 4)
+		(net_name "GND")
+		(layer "B.Cu")
+		(hatch edge 0.5)
+		(connect_pads
+			(clearance 0.5)
+		)
+		(min_thickness 0.25)
+		(filled_areas_thickness no)
+		(fill yes
+			(thermal_gap 0.5)
+			(thermal_bridge_width 0.5)
+		)
+		(polygon
+			(pts
+				(xy 153.543 54.864) (xy 171.704 54.61) (xy 171.577 83.185) (xy 150.769369 83.185) (xy 151.00731 57.963173)
+			)
+		)
+	)
 	(embedded_fonts no)

Commit message: trilhas modificado e nomes retirados
Other:
- board text added: "5V"
- board text added: "RX"
- board text removed: "Serial-arduino -> esp32 16/02/2026 Versão 1"
